File: ECAD/PmodADC/PmodADC.sch (KiCad schematic (older format))
At the start: 140 parts, among them J1 AudioIn, J2 Shield, J3 Pmod, J4 AudioOut, SW1 Bypass, SW2 Bypass, U1 74VHCT595BQ-Q100, U10 LM337_SOT223, U11 TLV172IDCK, U12 74VHCT595BQ-Q100, U13 74VHCT595BQ-Q100, U14 74AHCV541ABQ, U15 74AHCV541ABQ, U16 LF398_SOIC8, U17 TLV172IDCK, U18 TLV172IDCK, U19 LMV7235, U2 74VHCT595BQ-Q100, U3 MC34063AD, U4 MC34063AD, U5 74AHCV541ABQ, U6 74AHCV541ABQ, U8 L7805, U9 LM317_SOT-223

Commit message: Reworked Power Scheme
Parts:
- removed NT1: AGND, NetTie:NetTie-2_SMD_Pad2.0mm, symbol Device:Net-Tie_2
- added C15, C42: 100n, Capacitor_SMD:C_0402_1005Metric, symbol Device:C_Small
- added C19, C41: 1u, Capacitor_SMD:C_0402_1005Metric, symbol Device:C_Small
- added R67, R68, R69, R70: 100R, Resistor_SMD:R_0402_1005Metric, symbol Device:R_Small
- C25, C6: value 100n -> 1u
- C4: value 120pf -> 470p
- R4, R6: value 10K -> TODO
- R5, R7: value 56K -> TODO
Connections:
- net labels removed: GNDA
- wire segments 571 -> 590
Other:
- note added: "TODO: \n Raise Switchmode V's to 12V"
- note added: "Vin -> +12V Boost Pre-Regulator"
- note added: "Vin -> -12V Inverter"
- note removed: "TODO: \n Raise Switchmode V's to 12V\n Get rid of 5V seperation, AGND seperation.\n Maybe extra filtering on shift-registers.\n"
- note removed: "Vin -> +9V Boost Pre-Regulator"
- note removed: "Vin -> -9V Inverter"

Commit message: PCB v0.0 Done.
Parts:
- added C43, C44: 0u1, Capacitor_SMD:C_0402_1005Metric, symbol Device:C_Small
- added JP1, JP3: BitSelect, Jumper:SolderJumper-3_P1.3mm_Open_RoundedPad1.0x1.5mm, symbol Jumper:SolderJumper_3_Bridged12
- added JP2: Bypass, Jumper:SolderJumper-3_P1.3mm_Open_RoundedPad1.0x1.5mm, symbol Jumper:SolderJumper_3_Bridged12
- added JP4: Vref_Feedback, Jumper:SolderJumper-3_P1.3mm_Open_RoundedPad1.0x1.5mm, symbol Jumper:SolderJumper_3_Bridged12
- added R71, R72, R75, R76: 20K 0.1%, Resistor_SMD:R_0402_1005Metric, symbol Device:R_Small
- added R73, R74, R77, R78: 10K 0.1%, Resistor_SMD:R_0402_1005Metric, symbol Device:R_Small
- added TP10: S&H, TestPoint:TestPoint_Pad_D1.0mm, symbol Connector:TestPoint
- added TP11: S&H_o, TestPoint:TestPoint_Pad_D1.0mm, symbol Connector:TestPoint
- added TP12, TP15, TP19, TP4: GND, TestPoint:TestPoint_Pad_D1.0mm, symbol Connector:TestPoint
- added TP13, TP5: DAC, TestPoint:TestPoint_Pad_D1.0mm, symbol Connector:TestPoint
- added TP14: OUT1, TestPoint:TestPoint_Pad_D1.0mm, symbol Connector:TestPoint
- added TP16: OUT2, TestPoint:TestPoint_Pad_D1.0mm, symbol Connector:TestPoint
- added TP18: OUT, TestPoint:TestPoint_Pad_D1.0mm, symbol Connector:TestPoint
- added TP6: PREA, TestPoint:TestPoint_Pad_D1.0mm, symbol Connector:TestPoint
- added TP7: IN, TestPoint:TestPoint_Pad_D1.0mm, symbol Connector:TestPoint
- added TP9: S&H_i, TestPoint:TestPoint_Pad_D1.0mm, symbol Connector:TestPoint
- added U7: MAX6071BAUT50+T, Package_TO_SOT_SMD:SOT-23-6, symbol MAX6071:MAX6071
- C10, C13, C14, C15, C20, C21, C22, C23, C24, C26, C28, C29, C3, C35, C36, C38, C39, C40, C42, C5, C7, C9: value 100n -> 0u1
- C11: value 1000uF -> 1000u
- C12: value 1000uf -> 1000u
- C31, C33: value 100nf -> 0u1
- C8: value 470pf -> 470p
- D3: value LED -> Green
- J2: value Shield -> LeaderTech SMS405; footprint (none) -> Leader_SMS405:Leader_SMS405
- R4, R6: value TODO -> 12K
- R5, R7: value TODO -> 1K5
- R66: footprint Resistor_SMD:R_0603_1608Metric -> Resistor_SMD:R_0402_1005Metric
Connections:
- net +5V: now also U6.2 (A0); no longer C10.1, C28.1, C29.1, C9.1, U14.20 (VCC), U15.20 (VCC), U5.20 (VCC), U6.20 (VCC)
- net +9V: now also C43.1, U7.3 (EN), U7.4 (IN)
- net GND: now also C43.2, C44.2, TP12.1, TP15.1, TP19.1, TP4.1, U7.1 (GNDF), U7.2 (GNDS); no longer U15.4 (A2), U15.5 (A3), U6.2 (A0), U6.4 (A2), U6.5 (A3)
- net S&H: now also TP10.1
- net at TP1.1, U19.3 (+): now also JP2.2 (C); no longer U16.5
- net at TP2.1, U19.4 (-): now also JP1.2 (C), TP5.1; no longer R21.1, R32.2
- net at J1.T, SW1.3 (C), U11.1 (+): now also TP7.1
- net at J4.T, SW2.2 (B): now also TP18.1
- net at SW1.2 (B), U16.3 (I): now also JP2.3 (B), TP9.1
- net at R53.1, R64.2: now also JP3.3 (B), R77.1; no longer U17.1 (+)
- net at C37.2, SW2.3 (C), U17.3 (-)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: now also TP14.1
- net at SW2.1 (A), U18.3 (-), U18.4: now also TP16.1
- net at C27.1, R39.2, R40.1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: now also TP6.1
- net at U2.4 (QE): now also U6.5 (A3)
- net at U2.5 (QF): now also U6.4 (A2)
- net at U6.15 (Y3): now also R71.2
- net at U6.16 (Y2): now also R72.2
- net Vref_Sense: now reaches U6.18 (Y0)
- net Vref_Sense: now also JP4.3 (B)
- net at U13.4 (QE): now also U15.5 (A3)
- net at U13.5 (QF): now also U15.4 (A2)
- net at U15.15 (Y3): now also R75.2
- net at U15.16 (Y2): now also R76.2
- new net: JP2.1 (A), TP11.1, U16.5
- new net: JP3.2 (C), TP13.1, U17.1 (+)
- new net: JP1.3 (B), R21.1, R32.2, R73.1
- new net: R71.1, R73.2, R74.1
- new net: JP1.1 (A), R72.1, R74.2
- new net: JP4.2 (C), U7.5 (OUTS)
- new net: R75.1, R77.2, R78.1
- new net: JP3.1 (A), R76.1, R78.2
- new net Vref_5V: C10.1, C28.1, C29.1, C44.1, C9.1, JP4.1 (A), U14.20 (VCC), U15.20 (VCC), U5.20 (VCC), U6.20 (VCC), U7.6 (OUTF)
- no-connect marks 25 -> 15
Other:
- note added: "5V Ref"
- note added: "Note [1]: 12 or 14 bit dac. \nTo select 12 bit operation DNS last 4 resistors and use jumper\nto bypass them."
- note added: "Note [2]: 5V Ref Compensation:\nNot sure if good idea to include buffer\nin feedback path of 5V reference. Use jumper\nto select."
- note added: "See Note [1] for bit select"
- note removed: "TODO: \n Raise Switchmode V's to 12V"
- note removed: "https://www.mouser.ch/ProductDetail/LeaderTech/SMS-406C?qs=u16ybLDytRYS9HBi0epR5A%3D%3D"
- moved on the sheet: J2, SW1A, SW1B

Commit message: Quickfix PCB v0.1
Parts:
- removed C27, C37: 10u, Capacitor_SMD:C_0805_2012Metric, symbol Device:C_Small
- added C27, C37: 10u, Capacitor_THT:CP_Radial_D5.0mm_P2.00mm, symbol Device:CP_Small
- added C45: 1u, Capacitor_SMD:C_0402_1005Metric, symbol Device:C_Small
- added C46: 0u1, Capacitor_SMD:C_0402_1005Metric, symbol Device:C_Small
- added R79: 100R, Resistor_SMD:R_0402_1005Metric, symbol Device:R_Small
- added U20: 74AHCT541BQ,115, SOT764-1_DHVQFN20:SOT764-1_DHVQFN20, symbol 74xx:74HCT541
- U1, U12, U13, U2: value 74VHCT595BQ-Q100 -> 74VHC595BQ,115
Connections:
- net +5V: now also R79.1
- net ADC_C: now also U20.17 (Y1); no longer J3.3 (Pin_3)
- net ADC_L: now also U20.18 (Y0); no longer J3.1 (Pin_1)
- net ADC_S: now also U20.16 (Y2); no longer J3.5 (Pin_5)
- net DAC_C: now also U20.14 (Y4); no longer J3.4 (Pin_4)
- net DAC_L: now also U20.15 (Y3); no longer J3.2 (Pin_2)
- net DAC_S: now also U20.13 (Y5); no longer J3.6 (Pin_6)
- net GND: now also C45.2, C46.2, U20.1 (G1), U20.10 (GND), U20.19 (G2), U20.9 (A7)
- net S&H: now also U20.12 (Y6); no longer J3.7 (Pin_7)
- net at R37.1, U11.4: now also C27.1
- net at SW2.3 (C), TP14.1, U17.3 (-)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: now also C37.1
- net at RV3.1: now also C37.2
- net at R39.2, R40.1, SW1.1 (A)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: now also C27.2
- net COMP renamed COMP_3V
- new net: C45.1, C46.1, R79.2, U20.20 (VCC)
- new net ADC_C_3V: J3.3 (Pin_3), U20.3 (A1)
- new net ADC_L_3V: J3.1 (Pin_1), U20.2 (A0)
- new net ADC_S_3V: J3.5 (Pin_5), U20.4 (A2)
- new net DAC_C_3V: J3.4 (Pin_4), U20.6 (A4)
- new net DAC_L_3V: J3.2 (Pin_2), U20.5 (A3)
- new net DAC_S_3V: J3.6 (Pin_6), U20.7 (A5)
- new net S&H_3V: J3.7 (Pin_7), U20.8 (A6)
- no-connect marks 15 -> 16
Other:
- moved on the sheet: J3

Commit message: Added TODOs
Parts:
- added C?: 1n (C0G), symbol Device:C_Small
- added C? (x2): 0u1, Capacitor_SMD:C_0402_1005Metric, symbol Device:C_Small
- added R?: 6K8, symbol Device:R_Small
- added U?: TLV172IDCK, Package_TO_SOT_SMD:SOT-353_SC-70-5, symbol Amplifier_Operational:TLV172IDCK
Connections:
- net +9V: now also C?.2, U?.5 (V+)
- net -9V: now also C?.2, U?.2 (V-)
- net GND: now also C?.1, C?.1, C?.2
- net at SW1.3 (C), TP7.1, U11.1 (+): now also C?.1, R?.1; no longer J1.T
- new net: R?.2, U?.3 (-), U?.4
- new net: J1.T, U?.1 (+)
Other:
- note added: "AUDIO PREAMP + FILTER"
- note added: "TODO:\n Overall: \n Decide if to keep DAC\n If yes, add output Filter\n Different/Second Audio interface? (Mic, usw?)\n \n Fix:\n Fix PMOD Interface...?..!...\n Fix 5V Ref.\n\n Analog Performance\n Decide of use different 5v DAC buffer?\n Re-evalute Comparator\n if S&H needs offset adj, small SMD poti\n Decide if keep VREF feedback through buffer?\n \n Power Supply\n Change lm317 Rs to E12\n Fix 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"
- note added: "f_c = 23khz"
- note removed: "AUDIO PREAMP"
- moved on the sheet: C17, C21, C23, C24, C27, C30, C31, C32, C33, C34, C40, JP2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

Commit message: Finished Schematic Design
Parts:
- removed C1, C2: 100u, Capacitor_SMD:CP_Elec_8x6.5, symbol Device:CP_Small
- removed C11, C12: 1000u, Capacitor_SMD:CP_Elec_10x10.5, symbol Device:CP_Small
- removed C13, C14, C20, C21, C22, C3, C5: 0u1, Capacitor_SMD:C_0603_1608Metric, symbol Device:C_Small
- removed C16, C17, C18: 10u, Capacitor_SMD:CP_Elec_6.3x7.7, symbol Device:CP_Small
- removed C23, C24, C26, C28, C29, C35, C36, C38, C39, C42, C? (x2): 0u1, Capacitor_SMD:C_0402_1005Metric, symbol Device:C_Small
- removed C25, C41: 1u, Capacitor_SMD:C_0402_1005Metric, symbol Device:C_Small
- removed C27, C37: 10u, Capacitor_THT:CP_Radial_D5.0mm_P2.00mm, symbol Device:CP_Small
- removed C4, C8: 470p, Capacitor_SMD:C_0603_1608Metric, symbol Device:C_Small
- removed C?: 1n (C0G), symbol Device:C_Small
- removed D1, D2: 1N5819, Diode_SMD:D_SOD-123F, symbol Device:D_Schottky_Small
- removed D3: Green, Diode_SMD:D_0603_1608Metric, symbol Device:LED_Small
- removed J1: AudioIn, Jack_3.5mm_PJ-313D-6A:PJ-313D-6A, symbol Connector:AudioJack2
- removed J4: AudioOut, Jack_3.5mm_PJ-313D-6A:PJ-313D-6A, symbol Connector:AudioJack2
- removed JP1, JP3: BitSelect, Jumper:SolderJumper-3_P1.3mm_Open_RoundedPad1.0x1.5mm, symbol Jumper:SolderJumper_3_Bridged12
- removed JP2: Bypass, Jumper:SolderJumper-3_P1.3mm_Open_RoundedPad1.0x1.5mm, symbol Jumper:SolderJumper_3_Bridged12
- removed JP4: Vref_Feedback, Jumper:SolderJumper-3_P1.3mm_Open_RoundedPad1.0x1.5mm, symbol Jumper:SolderJumper_3_Bridged12
- removed L1, L2: 22uH 800mA, Inductor_SMD:L_Taiyo-Yuden_MD-4040, symbol Device:L
- removed R1, R2: 0R33 / 0.5W, Resistor_SMD:R_1210_3225Metric, symbol Device:R_Small
- removed R3: 180R, Resistor_SMD:R_0603_1608Metric, symbol Device:R_Small
- removed R33, R34, R5, R7: 1K5, Resistor_SMD:R_0603_1608Metric, symbol Device:R_Small
- removed R35, R36: 240R, Resistor_SMD:R_0603_1608Metric, symbol Device:R_Small
- removed R37: 100R, Resistor_SMD:R_0603_1608Metric, symbol Device:R_Small
- removed R38, R39, R40: 10K, Resistor_SMD:R_0603_1608Metric, symbol Device:R_Small
- removed R4, R6: 12K, Resistor_SMD:R_0603_1608Metric, symbol Device:R_Small
- removed R41, R42, R43, R44, R45, R46, R47, R48, R49, R50, R51, R52, R53, R75, R76: 20K 0.1%, Resistor_SMD:R_0402_1005Metric, symbol Device:R_Small
- removed R54, R55, R56, R57, R58, R59, R60, R61, R62, R63, R64, R77, R78: 10K 0.1%, Resistor_SMD:R_0402_1005Metric, symbol Device:R_Small
- removed R66: 10K, Resistor_SMD:R_0402_1005Metric, symbol Device:R_Small
- removed R69, R70, R79: 100R, Resistor_SMD:R_0402_1005Metric, symbol Device:R_Small
- removed R8: 22K, Resistor_SMD:R_0603_1608Metric, symbol Device:R_Small
- removed R?: 6K8, symbol Device:R_Small
- removed RV1: 47K, Bourns_3362P:Bourns_3362P, symbol Device:R_Variable
- removed RV3: 20K, Bourns_3362P:Bourns_3362P, symbol Device:R_POT
- removed SW1, SW2: Bypass, DPDT_5.6mm_2.5mm_SMD:DPDT_5.6mm_2.5mm_SMD, symbol Switch:SW_DPDT_x2
- removed TP13: DAC, TestPoint:TestPoint_Pad_D1.0mm, symbol Connector:TestPoint
- removed TP14: OUT1, TestPoint:TestPoint_Pad_D1.0mm, symbol Connector:TestPoint
- removed TP16: OUT2, TestPoint:TestPoint_Pad_D1.0mm, symbol Connector:TestPoint
- removed TP18: OUT, TestPoint:TestPoint_Pad_D1.0mm, symbol Connector:TestPoint
- removed TP19: GND, TestPoint:TestPoint_Pad_D1.0mm, symbol Connector:TestPoint
- removed TP3: Comp, TestPoint:TestPoint_Pad_D1.0mm, symbol Connector:TestPoint
- removed TP6: PREA, TestPoint:TestPoint_Pad_D1.0mm, symbol Connector:TestPoint
- removed TP7: IN, TestPoint:TestPoint_Pad_D1.0mm, symbol Connector:TestPoint
- removed U10: LM337_SOT223, Package_TO_SOT_SMD:SOT-223-3_TabPin2, symbol Regulator_Linear:LM337_SOT223
- removed U11, U17, U18, U?: TLV172IDCK, Package_TO_SOT_SMD:SOT-353_SC-70-5, symbol Amplifier_Operational:TLV172IDCK
- removed U12, U13: 74VHC595BQ,115, SOT763-1_DHVQFN16:SOT763-1_DHVQFN16, symbol 74xx:74HC595
- removed U14, U15: 74AHCV541ABQ, SOT764-1_DHVQFN20:SOT764-1_DHVQFN20, symbol 74xx:74LS541
- removed U19: LMV7235, Package_TO_SOT_SMD:SOT-353_SC-70-5, symbol LMV7235:LMV7235
- removed U3, U4: MC34063AD, Package_SO:SOIC-8_3.9x4.9mm_P1.27mm, symbol Regulator_Switching:MC34063AD
- removed U8: L7805, Package_TO_SOT_SMD:SOT-223, symbol Regulator_Linear:L7805
- removed U9: LM317_SOT-223, Package_TO_SOT_SMD:SOT-223-3_TabPin2, symbol PmodADC-rescue:LM317_SOT-223-Regulator_Linear
- added C? (x7): 10u, symbol Device:C_Small
- added C?: DNS, Capacitor_SMD:C_0402_1005Metric, symbol Device:C_Small
- added C? (x6): 1u, symbol Device:C_Small
- added C? (x2): 10u, symbol Device:CP1_Small
- added C? (x4): 0u1, symbol Device:C_Small
- added C?: 0u1, Capacitor_SMD:C_0402_1005Metric, symbol Device:C_Small
- added C?: 4u7, symbol Device:C_Small
- added C?: 1u, Capacitor_SMD:C_0402_1005Metric, symbol Device:C_Small
- added C?: 10n C0G, symbol Device:C_Small
- added C?: 4n7 C0G, symbol Device:C_Small
- added C?: 4n7, symbol Device:C_Small
- added C?: 0u22, symbol Device:C_Small
- added D?: SL03, symbol Device:D_Schottky_Small
- added FB? (x4): 100R/100MHz, symbol Device:Ferrite_Bead_Small
- added J?: AudioIn, Jack_3.5mm_PJ-313D-6A:PJ-313D-6A, symbol Connector:AudioJack3
- added J?: AudioIn, Connector_PinHeader_2.54mm:PinHeader_1x02_P2.54mm_Vertical, symbol Connector_Generic:Conn_01x02
- added JP?: byp, Resistor_SMD:R_0402_1005Metric, symbol Device:Jumper_NO_Small
- added JP? (x3): disc, Resistor_SMD:R_0402_1005Metric, symbol Device:Jumper_NC_Small
- added JP?: Jumper, Resistor_SMD:R_0402_1005Metric, symbol Device:Jumper_NC_Small
- added JP?: DNS, Resistor_SMD:R_0402_1005Metric, symbol Device:Jumper_NO_Small
- added JP?: DI, Resistor_SMD:R_0402_1005Metric, symbol Device:Jumper_NO_Small
- added JP?: Normal, Resistor_SMD:R_0402_1005Metric, symbol Device:Jumper_NC_Small
- added L?: 100n, symbol Device:L_Small
- added L? (x2): 22uH, 300mA, symbol Device:L_Small
- added R?: 100k, Resistor_SMD:R_0402_1005Metric, symbol Device:R_Small
- added R? (x3): 15k, Resistor_SMD:R_0402_1005Metric, symbol Device:R_Small
- added R? (x2): 47k, Resistor_SMD:R_0402_1005Metric, symbol Device:R_Small
- added R?: 50k Log, symbol Device:R_Variable
- added R?: 5k, symbol Device:R_Small
- added R?: 68k, symbol Device:R_Small
- added R?: 5k6, symbol Device:R_Small
- added R?: 10R, symbol Device:R_Small
- added R? (x2): 1k2, symbol Device:R_Small
- added R?: 120k, symbol Device:R_Small
- added R?: 560k, symbol Device:R_Small
- added R?: 100R, Resistor_SMD:R_0402_1005Metric, symbol Device:R_Small
- added R? (x2): 20k, symbol Device:R_Small
- added R?: 33k, symbol Device:R_Small
- added R?: 10k, symbol Device:R_Small
- added RV?: 1K, symbol Device:R_POT
- added TP? (x2): IN, TestPoint:TestPoint_Pad_D1.0mm, symbol Connector:TestPoint
- added TP?: GND, TestPoint:TestPoint_Pad_D1.0mm, symbol Connector:TestPoint
- added U? (x2): LDK320AM-R, symbol LDK220_LDK320:LDK320_SOT32-5
- added U?: SN74LVC1G17DCK, Package_TO_SOT_SMD:SOT-353_SC-70-5, symbol 74xGxx:74LVC1G17
- added U? (x3): OPA1602, symbol Amplifier_Operational:OPA1602
- added U?: MIC5270, symbol MIC5270:MIC5270
- added U?: TLV61046ADB, Package_TO_SOT_SMD:SOT-23-6, symbol Regulator_Switching:TLV61046ADB
- added U?: TPS63700, Package_SON:VSON-10-1EP_3x3mm_P0.5mm_EP1.65x2.4mm_ThermalVias, symbol TPS63700:TPS63700
- added U?: LT1711xMS8, Package_SO:MSOP-8_3x3mm_P0.65mm, symbol Comparator:LT1711xMS8
- C34: value 10nF -> 10nF C0G
- RV2: footprint Bourns_3362P:Bourns_3362P -> (none)
- U7: value MAX6071BAUT50+T -> REF3450
Connections:
- net DAC_L is gone; now on net S&H: U20.15 (Y3)
- net +3V3: now also J3.11 (Pin_11), J3.12 (Pin_12), C?.1, C?.1, C?.1, L?.1, R?.1, U?.4 (EN), U?.5 (IN), U?.5 (VCC), U?.6 (VI); no longer J3.10 (Pin_10), J3.9 (Pin_9)
- net +5V: now also C?.1, FB?.1, FB?.1, FB?.1, JP?.2, L?.1, U?.1 (V+); no longer R67.1, R68.1, U6.2 (A0)
- net +9V: now also C?.1, C?.1, JP?.2, U?.8 (V+)
- net COMP_3V: now also U?.4
- net GND: now also J3.10 (Pin_10), J3.9 (Pin_9), U20.7 (A5), U20.8 (A6), U6.2 (A0), C?.1, C?.1, C?.1, C?.1, C?.1, C?.1, C?.1, C?.1, C?.1, C?.1, C?.2, C?.2, C?.2, C?.2, C?.2, C?.2, C?.2, C?.2, C?.2, C?.2, C?.2, C?.2, C?.2, C?.2, J?.1 (Pin_1), J?.S, L?.2, R?.1, R?.1, R?.2, R?.2, R?.2, R?.2, R?.2, TP?.1, U?.11 (PAD), U?.2 (GND), U?.2 (GND), U?.2 (GND), U?.2 (GND), U?.2 (GND), U?.3 (GND), U?.4 (V-), U?.6 (GND), U?.7 (PS_GND); no longer J3.11 (Pin_11), J3.12 (Pin_12), U20.10 (GND)
- net S&H: no longer U20.12 (Y6)
- net S&H_3V: now also U20.5 (A3); no longer U20.8 (A6)
- net Vref_5V: now also C?.1, C?.1, FB?.1, R?.2; no longer C44.1, U7.6 (OUTF)
- net at TP1.1: now also JP?.1, JP?.2, U?.2 (+)
- net at TP2.1, TP5.1: now also R72.1, R74.2, C?.1, U?.3 (-)
- net at TP9.1, U16.3 (I): now also JP?.2, JP?.2, JP?.2
- net at TP11.1, U16.5: now also JP?.1
- net at C45.1, C46.1, U20.20 (VCC): now also R?.2
- net at U7.5 (OUTS): now also C44.1, U7.6 (OUTF), FB?.2
- net -9V renamed -5V
- net -5V: now also C?.2, C?.2, JP?.2, U?.4 (V-)
- net DAC_C renamed COMP_L
- net DAC_C_3V: no longer names the net of J3.4 (Pin_4)
- net DAC_C_3V: no longer U20.6 (A4)
- net DAC_L_3V: no longer names the net of J3.2 (Pin_2)
- net DAC_L_3V: no longer U20.5 (A3)
- net DAC_S: no longer names the net of U20.13 (Y5)
- net DAC_S_3V renamed COMP_L_3V
- net COMP_L_3V: now also U20.6 (A4); no longer U20.7 (A5)
- net Vref_Sense: no longer names the net of U6.18 (Y0)
- new net: FB?.2, R68.1
- new net: C?.1, J?.2 (Pin_2), J?.T, JP?.1, TP?.1
- new net: C?.1, C?.2, C?.2, R?.1, U?.1 (IN), U?.1 (IN), U?.3 (EN), U?.3 (EN), U?.5 (VOUT)
- new net: R?.1, R?.2, U?.4 (ADJ/NC) (x2)
- new net: C?.1, JP?.1, R?.1, U?.5 (OUT) (x2)
- new net: FB?.2, R67.1
- new net: R?.1, R?.2, U?.1
- new net: R?.2, R?.2, U?.2 (-)
- new net: C?.2, R?.1, U?.5 (+)
- new net: C?.1, C?.2, U?.6 (-), U?.7
- new net: R?.1, R?.2, U?.3 (ADJ/NC)
- new net: C?.2, JP?.1, R?.1, U?.4 (OUT)
- new net: C?.1, C?.1, D?.2 (A), R?.1, U?.5 (IN), U?.8 (OUT)
- new net: L?.2, U?.1 (SW)
- new net: R?.1, R?.2, U?.3 (FB)
- new net: C?.2, U?.1 (COMP)
- new net: C?.2, R?.2, U?.10 (VREF)
- new net: C?.2, R?.2, U?.3 (VIN), U?.4 (EN)
- new net: D?.1 (K), L?.1, U?.6 (SW)
- new net: R?.1, R?.2, U?.9 (FB)
- new net: C?.2, R?.1, R?.2
- new net: C?.1, JP?.1, RV?.2, TP?.1
- new net: R?.1, R?.2
- new net: FB?.2, R?.1
- new net: R?.1, RV?.1
- new net: R?.2, RV?.3
- new net +5VA: C?.2, L?.2
- new net COMP: U?.2, U?.7 (Q)
- new net COMP_L_5v: U?.5 (LATCH)
- new net DI: C?.2, JP?.1, JP?.2, R?.1, U?.3 (+)
- no-connect marks 16 -> 12
Other:
- note added: "+3V3 -> +10V Boost"
- note added: "+3V3 -> -6V Inverter"
- note added: "+9V Linear Regulator"
- note added: "-5V Linear Regulator"
- note added: "1x-11x Amplification"
- note added: "20khz Sallen-Key LP"
- note added: "Aprox. +/- 5mV \nBias Point Adj."
- note added: "Biasing"
- note added: "Bypass \nfor testing"
- note added: "Gain"
- note added: "Input"
- note added: "Input + Signal Conditioning"
- note added: "Input Levelshift"
- note added: "Input voltage range \n 100mV beyond supply."
- note added: "Note: Actual Vout \naprox 10.5V"
- note added: "Output Levelshift"
- note added: "Populate either \nC/R or JP. (In case \nDC offs. becomes \na problem during \namplification)"
- note removed: "+/-9V Linear Regulator"
- note removed: "AUDIO OUTPUT STAGE"
- note removed: "AUDIO PREAMP + FILTER"
- note removed: "Hold Capacitor:\nTDK C1608C0G1E103J080AA"
- note removed: "Input voltage range \n 200mV beyond supply."
- note removed: "Note [1]: 12 or 14 bit dac. \nTo select 12 bit operation DNS last 4 resistors and use jumper\nto bypass them."
- note removed: "Note [2]: 5V Ref Compensation:\nNot sure if good idea to include buffer\nin feedback path of 5V reference. Use jumper\nto select."
- note removed: "See Note [1] for bit select"
- note removed: "Shield: ADC's DAC, S&H, \nComparator"
- note removed: "TODO:\n Overall: \n Decide if to keep DAC\n If yes, add output Filter\n Different/Second Audio interface? (Mic, usw?)\n \n Fix:\n Fix PMOD Interface...?..!...\n Fix 5V Ref.\n\n Analog Performance\n Decide of use different 5v DAC buffer?\n Re-evalute Comparator\n if S&H needs offset adj, small SMD poti\n Decide if keep VREF feedback through buffer?\n \n Power Supply\n Change lm317 Rs to E12\n Fix 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"
- note removed: "Vin -> +12V Boost Pre-Regulator"
- note removed: "Vin -> -12V Inverter"
- note removed: "f_c = 23khz"
- moved on the sheet: C10, C15, C19, C30, C31, C32, C33, C34, C40, C43, C44, C45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

Commit message: Added Footprints, fixedup Schematic, Cleanup
Parts:
- removed L?: 100n, symbol Device:L_Small
- removed TP1: S&H, TestPoint:TestPoint_Pad_D1.0mm, symbol Connector:TestPoint
- removed TP12, TP15, TP4, TP?: GND, TestPoint:TestPoint_Pad_D1.0mm, symbol Connector:TestPoint
- removed TP2: DAC, TestPoint:TestPoint_Pad_D1.0mm, symbol Connector:TestPoint
- removed U?: MIC5270, symbol MIC5270:MIC5270
- added FB5: 1K/100MHz, Inductor_SMD:L_0402_1005Metric, symbol Device:Ferrite_Bead_Small
- added U10: MIC5270BM5, Package_TO_SOT_SMD:SOT-23-5, symbol MIC5270:MIC5270
- C1: renamed from C?; footprint (none) -> Capacitor_SMD:C_0805_2012Metric
- C11, C17, C18, C2, C20, C27, C8: renamed from C?; footprint (none) -> Capacitor_SMD:C_1206_3216Metric
- C12, C13, C14, C22, C25, C28, C29, C3, C35, C36, C4, C5: renamed from C?; footprint (none) -> Capacitor_SMD:C_0402_1005Metric
- C16, C26: renamed from C?; footprint (none) -> Capacitor_THT:CP_Radial_D4.0mm_P1.50mm
- C23, C24: renamed from C?; footprint (none) -> Capacitor_SMD:C_0603_1608Metric
- C30, C31, C32, C33: footprint Capacitor_SMD:C_0603_1608Metric -> Capacitor_SMD:C_0402_1005Metric
- D1: renamed from D?; footprint (none) -> Diode_SMD:D_SMF
- FB1, FB2, FB3, FB4: renamed from FB?; value 100R/100MHz -> 1K/100MHz; footprint (none) -> Inductor_SMD:L_0402_1005Metric
- L1, L2: renamed from L?; footprint (none) -> Inductor_SMD:L_Wuerth_MAPI-3020
- R1, R2, R3, R38, R39, R4, R41, R42, R43, R44, R5, R6: renamed from R?; footprint (none) -> Resistor_SMD:R_0402_1005Metric
- R40: renamed from R?; footprint (none) -> Potentiometer_THT:Potentiometer_Alps_RK09L_Single_Vertical
- R65: footprint Resistor_SMD:R_0603_1608Metric -> Resistor_SMD:R_0402_1005Metric
- RV1: renamed from RV?; footprint (none) -> Potentiometer_SMD:Potentiometer_Bourns_TC33X_Vertical
- RV2: footprint (none) -> Potentiometer_SMD:Potentiometer_Bourns_TC33X_Vertical
- U12: renamed from U?; footprint (none) -> Package_SO:VSSOP-8_3.0x3.0mm_P0.65mm
- U8, U9: renamed from U?; footprint (none) -> Package_TO_SOT_SMD:SOT-23-5
- gave numbers to parts that had none: 26
Connections:
- net COMP_L_5v is gone; now on net COMP_L: U13.5 (LATCH)
- net +5V: now also FB5.1; no longer C38.1, C40.1, U13.1 (V+)
- net +5VA: now also C38.1, C40.1, U13.1 (V+), FB5.2
- net GND: now also U20.10 (GND); no longer C10.2, C12.1, C13.1, C14.2, C17.2, C18.2, C20.1, C22.1, C24.1, C25.2, C27.2, C28.2, C29.1, C30.2, C31.2, C32.2, C33.2, C34.2, C35.2, C36.1, C37.2, C38.2, C40.2, C43.2, C44.2, C9.2, J1.1 (Pin_1), J2.1 (Shield), J3.10 (Pin_10), J4.S, R33.2, R35.2, R36.2, R38.2, R39.1, R44.1, R65.1, R9.2, U13.4 (V-), U13.6 (GND), U16.7 (T), U5.1 (G1), U5.10 (GND), U5.19 (G2), U6.1 (G1), U6.10 (GND), U6.19 (G2), U6.2 (A0), U6.3 (A1), U7.1 (GNDF), U7.2 (GNDS), U8.2 (GND), U9.2 (GND)
- net at R36.1, R37.2: now also U10.3 (ADJ/NC)
- net at C20.2, JP4.1, R37.1: now also U10.4 (OUT)
- net at C11.1, C14.1, D1.2 (A)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: now also U10.5 (IN)
- new net GNDA: C10.2, C12.1, C13.1, C14.2, C17.2, C18.2, C20.1, C22.1, C24.1, C25.2, C27.2, C28.2, C29.1, C30.2, C31.2, C32.2, C33.2, C34.2, C35.2, C36.1, C37.2, C38.2, C40.2, C43.2, C44.2, C9.2, J1.1 (Pin_1), J2.1 (Shield), J3.10 (Pin_10), J4.S, R33.2, R35.2, R36.2, R38.2, R39.1, R44.1, R65.1, R9.2, U10.2 (GND), U13.4 (V-), U13.6 (GND), U16.7 (T), U5.1 (G1), U5.10 (GND), U5.19 (G2), U6.1 (G1), U6.10 (GND), U6.19 (G2), U6.2 (A0), U6.3 (A1), U7.1 (GNDF), U7.2 (GNDS), U8.2 (GND), U9.2 (GND)
Other:
- note added: "Everything except Power\nSupply, Controls, and \nConnectors."
- note added: "GND and GNDA\nconnected on \nPmod host."
- moved on the sheet: C18, C22, C25, J3, JP3
