File: ECAD/PmodDAC/PmodDAC.kicad_pcb (KiCad board)
At the start: 4 copper layers, 28.6 x 80.6 mm, 122 parts, among them J1 AudioOut, J2 LeaderTech SMS405, J3 Pmod, J4 AudioOut, U1 74VHC595BQ,115, U10 MIC5270BM5, U11 OPA1656, U12 OPA1656, U2 74VHC595BQ,115, U20 74AHCT541BQ,115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

Commit message: Added DAC Production Files
Routing:
- net GNDA: track 191.7 -> 194.7 mm, vias 28 -> 46
- net -5V: track 65.3 -> 63.0 mm
- net Net-(J1-Pad2): track 38.2 -> 39.3 mm
