File: ECAD/PmodDAC/PmodDAC.sch (KiCad schematic (older format))
At the start: 122 parts, among them J1 AudioOut, J2 LeaderTech SMS405, J3 Pmod, J4 AudioOut, U1 74VHC595BQ,115, U10 MIC5270BM5, U11 OPA1656, U12 OPA1656, U2 74VHC595BQ,115, U20 74AHCT541BQ,115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

Commit message: Added DAC Production Files
Changed lines of the file:
@@
 encoding utf-8
 Sheet 1 1
-Title "PmodADC"
-Date "2020-10-12"
-Rev "v0.1"
+Title "PmodDAC"
+Date "2020-10-31"
+Rev "v0.2"
 Comp "Philipp Schilk"
 Comment1 ""
 Comment2 ""
 Comment3 ""
-Comment4 ""
+Comment4 "https://github.com/TheSchilk/PmodADC"
 $EndDescr
 $Comp
@@
 	1    0    0    -1
 $EndComp
-Text Notes 9650 5550 0    79   ~ 0
+Text Notes 9350 5500 0    79   ~ 0
 20khz Sallen-Key LP
 Connection ~ 11950 4000
@@
 Wire Wire Line
 	14300 4350 14750 4350
+Text Notes 11200 5500 0    79   ~ 0
+20khz Sallen-Key LP
 $EndSCHEMATC
